Commit message: learn: Test gazebo with urdf model also test inertia xacro

File: urdf/my_robot.urdf.xacro (robot description, xacro)
@@ -3,4 +3,5 @@
     <!-- Other xacro files -->
     <xacro:include filename="materials.urdf.xacro" />
+    <xacro:include filename="inertia.urdf.xacro" />
     <!-- Xacro properties -->
     <xacro:property name="radius" value="0.1" />
@@ -16,4 +17,11 @@
                 <material name="grey" />
             </visual>
+            <collision>
+                <geometry>
+                    <cylinder radius="${radius}" length="${length}" />
+                </geometry>
+                <origin xyz="0 0 0" rpy="1.57 0 0" />
+            </collision>
+            <xacro:cylinder_inertia mass="0.5" radius="${radius}" length="${length}"/>
         </link>
     </xacro:macro>
@@ -44,4 +52,11 @@
             <material name="green" />
         </visual>
+        <collision>
+            <geometry>
+                <box size="0.6 0.4 0.2" />
+            </geometry>
+            <origin xyz="0 0 0.1" rpy="0 0 0" />
+        </collision>
+        <xacro:box_inertia mass="5" x="0.6" y="0.4" z="0.2"/>
     </link>
     <link name="lidar_link">
@@ -62,4 +77,11 @@
             <material name="grey" />
         </visual>
+        <collision>
+            <geometry>
+                <sphere radius="${radius}" />
+            </geometry>
+            <origin xyz="0 0 0" rpy="0 0 0" />
+        </collision>
+        <xacro:sphere_inertia mass="0.2" radius="0.1"/>
     </link>
     <xacro:wheels prefix="left" />
@@ -71,3 +93,15 @@
     <xacro:continuous_joint prefix="base_left_wheel" parent="main_body_link" child="left_wheel_link" xyz="-0.15 0.225 0" rpy="0 0 0" axis="0 1 0"/>
     <xacro:continuous_joint prefix="base_right_wheel" parent="main_body_link" child="right_wheel_link" xyz="-0.15 -0.225 0" rpy="0 0 0" axis="0 1 0"/>
+    <!-- Gazebo Section -->
+    <gazebo>
+        <plugin
+            filename="gz-sim-diff-drive-system"
+            name="gz::sim::systems::DiffDrive">
+            <left_joint>base_left_wheel_joint</left_joint>
+            <right_joint>base_right_wheel_joint</right_joint>
+            <wheel_separation>0.45</wheel_separation>
+            <wheel_radius>0.1</wheel_radius>
+            <topic>cmd_vel</topic>
+        </plugin>
+    </gazebo>
 </robot>
