Commit message: feat: Add lidar sensor

File: learn_ros/description/urdf/robot.urdf.xacro (robot description, xacro)
@@ -75,5 +75,5 @@
         <collision>
             <geometry>
-                <box size="${radius_wheels*2} ${radius_wheels*2} ${length}" />
+                <cylinder radius="${radius_wheels}" length="${length}" />
             </geometry>
             <origin xyz="0 0 0" rpy="0 0 0" />
@@ -138,3 +138,40 @@
         </plugin>
     </gazebo>
+    <!-- Lidar sensor -->
+    <gazebo>
+        <plugin
+            filename="gz-sim-sensors-system"
+            name="gz::sim::systems::Sensors">
+            <render_engine>ogre2</render_engine>
+        </plugin>
+    </gazebo>
+    <gazebo reference="lidar_link">
+        <sensor name="gpu_lidar" type="gpu_lidar">
+            <pose relative_to="lidar_link">0 0 0 0 0 0</pose>
+            <topic>lidar</topic>
+            <update_rate>2</update_rate>
+            <lidar>
+                <scan>
+                    <horizontal>
+                        <samples>720</samples>
+                        <resolution>1</resolution>
+                        <min_angle>-3.14</min_angle>
+                        <max_angle>3.14</max_angle>
+                    </horizontal>
+                </scan>
+                <range>
+                    <min>0.01</min>
+                    <max>12.0</max>
+                    <resolution>0.005</resolution>
+                </range>
+                <noise>
+                    <type>gaussian</type>
+                    <mean>0.0</mean>
+                    <stddev>0.001</stddev>
+                </noise>
+            </lidar>
+            <always_on>1</always_on>
+            <visualize>1</visualize>
+        </sensor>
+    </gazebo>
 </robot>
