Commit message: feat: Add camera sensor

File: learn_ros/description/urdf/materials.urdf.xacro (robot description, xacro)
@@ -10,3 +10,6 @@
         <color rgba="1 1 1 1" />
     </material>
+    <material name="black">
+        <color rgba="0 0 0 1" />
+    </material>
 </robot>

File: learn_ros/description/urdf/robot.urdf.xacro (robot description, xacro)
@@ -65,4 +65,22 @@
             xyz="0 0 0.1" rpy="0 0 0"/>
     </link>
+    <link name="camera_link">
+        <visual>
+            <geometry>
+                <box size="0.025 0.025 0.025" />
+            </geometry>
+            <origin xyz="0 0 0" rpy="0 0 0" />
+            <material name="white" />
+        </visual>
+        <collision>
+            <geometry>
+                <box size="0.025 0.025 0.025" />
+            </geometry>
+            <origin xyz="0 0 0" rpy="0 0 0" />
+        </collision>
+        <xacro:solid_box_inertia
+            mass="0.01" x="0.025" y="0.025" z="0.025"
+            xyz="0 0 0" rpy="0 0 0"/>
+    </link>
     <link name="lidar_link">
         <visual>
@@ -105,4 +123,9 @@
         xyz="0 0 0.1" rpy="0 0 0"/>
     <xacro:fixed_joint
+        prefix="base_camera"
+        parent="main_body_link"
+        child="camera_link"
+        xyz="0.3125 0 0.1" rpy="0 0 0"/>
+    <xacro:fixed_joint
         prefix="base_lidar"
         parent="main_body_link"
@@ -113,5 +136,5 @@
         parent="main_body_link"
         child="caster_wheel_link"
-        xyz="0.2 0 -0.025" rpy="0 0 0" />
+        xyz="0.2 0 -${radius_caster_wheel}" rpy="0 0 0" />
     <xacro:continuous_joint
         prefix="base_left_wheel"
@@ -137,4 +160,26 @@
             <topic>cmd_vel</topic>
         </plugin>
+    </gazebo>
+    <!-- Camera sensor -->
+    <gazebo reference="camera_link">
+        <sensor name="camera" type="camera">
+            <pose relative_to="camera_link">0 0 0 0 0 0</pose>
+            <topic>camera</topic>
+            <update_rate>30.0</update_rate>
+            <camera>
+                <horizontal_fov>1.047</horizontal_fov>
+                <image>
+                    <width>640</width>
+                    <height>480</height>
+                    <format>R8G8B8</format>
+                </image>
+                <clip>
+                    <near>0.05</near>
+                    <far>8.0</far>
+                </clip>
+            </camera>
+            <always_on>1</always_on>
+            <visualize>1</visualize>
+        </sensor>
     </gazebo>
     <!-- Lidar sensor -->
